File: TSOC_GROVEY_ONE/TSOC_GROVEY_ONE.brd (EAGLE design)
At the start: 44.5 x 30.5 mm, 53 parts, among them J3 NO, J4 6p-2.54, U1 MIC5219 3.3V, U2 ATMEGA328, X1 16MHZ

Commit message: update to Rev 2.0
Parts:
- R10, R4, R5, R7, R8, R9: value 1K 1/10W -> 1K
Other:
- outline, holes or cut-outs redrawn
Changed lines of the file:
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@@
 <layer number="23" name="tOrigins" color="15" fill="1" visible="yes" active="yes"/>
 <layer number="24" name="bOrigins" color="15" fill="1" visible="yes" active="yes"/>
-<layer number="25" name="tNames" color="7" fill="1" visible="no" active="yes"/>
+<layer number="25" name="tNames" color="7" fill="1" visible="yes" active="yes"/>
 <layer number="26" name="bNames" color="7" fill="1" visible="yes" active="yes"/>
 <layer number="27" name="tValues" color="7" fill="1" visible="no" active="yes"/>
@@
 <attribute name="VALUE" x="42.926" y="24.257" size="0.889" layer="27" font="vector" ratio="11" rot="R270"/>
 </element>
-<element name="R9" library="Seeed-Resistor-2016" package="R0603" value="1K 1/10W" x="34.29" y="20.574" smashed="yes">
+<element name="R9" library="Seeed-Resistor-2016" package="R0603" value="1K" x="34.29" y="20.574" smashed="yes">
 <attribute name="NAME" x="33.528" y="19.939" size="0.8128" layer="25" font="vector" ratio="15" rot="R90"/>
-<attribute name="VALUE" value="1K 1/10W" x="33.274" y="19.431" size="0.4064" layer="27" font="vector"/>
-<attribute name="MPN" value="RC0603JR-071KL" x="34.29" y="20.574" size="1.778" layer="27" display="off"/>
-</element>
-<element name="R10" library="Seeed-Resistor-2016" package="R0603" value="1K 1/10W" x="34.29" y="23.622" smashed="yes" rot="R180">
+<attribute name="VALUE" value="2.2K" x="33.274" y="19.431" size="0.4064" layer="27" font="vector"/>
+<attribute name="MPN" value="RC0603JR-072K2L" x="34.29" y="20.574" size="1.778" layer="27" display="off"/>
+</element>
+<element name="R10" library="Seeed-Resistor-2016" package="R0603" value="1K" x="34.29" y="23.622" smashed="yes" rot="R180">
 <attribute name="NAME" x="32.766" y="24.257" size="0.8128" layer="25" font="vector" ratio="15" rot="R270"/>
-<attribute name="VALUE" value="1K 1/10W" x="35.306" y="24.765" size="0.4064" layer="27" font="vector" rot="R180"/>
-<attribute name="MPN" value="RC0603JR-071KL" x="34.29" y="23.622" size="1.778" layer="27" rot="R180" display="off"/>
-</element>
-<element name="R7" library="Seeed-Resistor-2016" package="R0603" value="1K 1/10W" x="34.29" y="10.16" smashed="yes">
+<attribute name="VALUE" value="2.2K" x="35.306" y="24.765" size="0.4064" layer="27" font="vector" rot="R180"/>
+<attribute name="MPN" value="RC0603JR-072K2L" x="34.29" y="23.622" size="1.778" layer="27" rot="R180" display="off"/>
+</element>
+<element name="R7" library="Seeed-Resistor-2016" package="R0603" value="1K" x="34.29" y="10.16" smashed="yes">
 <attribute name="NAME" x="33.528" y="9.525" size="0.8128" layer="25" font="vector" ratio="15" rot="R90"/>
-<attribute name="VALUE" value="1K 1/10W" x="33.274" y="9.017" size="0.4064" layer="27" font="vector"/>
-<attribute name="MPN" value="RC0603JR-071KL" x="34.29" y="10.16" size="1.778" layer="27" display="off"/>
-</element>
-<element name="R8" library="Seeed-Resistor-2016" package="R0603" value="1K 1/10W" x="34.29" y="13.208" smashed="yes" rot="R180">
+<attribute name="VALUE" value="2.2K" x="33.274" y="9.017" size="0.4064" layer="27" font="vector"/>
+<attribute name="MPN" value="RC0603JR-072K2L" x="34.29" y="10.16" size="1.778" layer="27" display="off"/>
+</element>
+<element name="R8" library="Seeed-Resistor-2016" package="R0603" value="1K" x="34.29" y="13.208" smashed="yes" rot="R180">
 <attribute name="NAME" x="33.528" y="12.573" size="0.8128" layer="25" font="vector" ratio="15" rot="R90"/>
-<attribute name="VALUE" value="1K 1/10W" x="35.306" y="14.351" size="0.4064" layer="27" font="vector" rot="R180"/>
-<attribute name="MPN" value="RC0603JR-071KL" x="34.29" y="13.208" size="1.778" layer="27" rot="R180" display="off"/>
+<attribute name="VALUE" value="2.2K" x="35.306" y="14.351" size="0.4064" layer="27" font="vector" rot="R180"/>
+<attribute name="MPN" value="RC0603JR-072K2L" x="34.29" y="13.208" size="1.778" layer="27" rot="R180" display="off"/>
 </element>
 <element name="R3" library="Seeed-Resistor-2016" package="R0603" value="2.2K" x="9.906" y="9.906" smashed="yes" rot="R180">
@@
 <attribute name="MPN" value="RC0603JR-072K2L" x="9.906" y="6.858" size="1.778" layer="27" display="off"/>
 </element>
-<element name="R5" library="Seeed-Resistor-2016" package="R0603" value="1K 1/10W" x="9.906" y="21.082" smashed="yes">
+<element name="R5" library="Seeed-Resistor-2016" package="R0603" value="1K" x="9.906" y="21.082" smashed="yes">
 <attribute name="NAME" x="10.668" y="21.717" size="0.8128" layer="25" font="vector" ratio="15" rot="R270"/>
-<attribute name="VALUE" value="1K 1/10W" x="8.89" y="19.939" size="0.4064" layer="27" font="vector"/>
-<attribute name="MPN" value="RC0603JR-071KL" x="9.906" y="21.082" size="1.778" layer="27" display="off"/>
-</element>
-<element name="R4" library="Seeed-Resistor-2016" package="R0603" value="1K 1/10W" x="9.906" y="18.034" smashed="yes" rot="R180">
+<attribute name="VALUE" value="2.2K" x="8.89" y="19.939" size="0.4064" layer="27" font="vector"/>
+<attribute name="MPN" value="RC0603JR-072K2L" x="9.906" y="21.082" size="1.778" layer="27" display="off"/>
+</element>
+<element name="R4" library="Seeed-Resistor-2016" package="R0603" value="1K" x="9.906" y="18.034" smashed="yes" rot="R180">
 <attribute name="NAME" x="10.668" y="18.923" size="0.8128" layer="25" font="vector" ratio="15" rot="R270"/>
-<attribute name="VALUE" value="1K 1/10W" x="10.922" y="19.177" size="0.4064" layer="27" font="vector" rot="R180"/>
-<attribute name="MPN" value="RC0603JR-071KL" x="9.906" y="18.034" size="1.778" layer="27" rot="R180" display="off"/>
+<attribute name="VALUE" value="2.2K" x="10.922" y="19.177" size="0.4064" layer="27" font="vector" rot="R180"/>
+<attribute name="MPN" value="RC0603JR-072K2L" x="9.906" y="18.034" size="1.778" layer="27" rot="R180" display="off"/>
 </element>
 <element name="FID4" library="TSOC-ESP8266-BASE" package="MICRO-FIDUCIAL" value="FIDUCIALUFIDUCIAL" x="40.64" y="2.032"/>
@@
 <wire x1="22.86" y1="13.462" x2="23.368" y2="13.97" width="0.6096" layer="16"/>
 <wire x1="23.368" y1="13.97" x2="26.162" y2="13.97" width="0.6096" layer="16"/>
-<wire x1="12.446" y1="13.8684" x2="12.446" y2="13.81126875" width="0.1778" layer="1"/>
 <wire x1="12.446" y1="13.6906" x2="12.446" y2="13.716" width="0.1778" layer="1"/>
-<wire x1="12.446" y1="13.716" x2="12.446" y2="13.81126875" width="0.1778" layer="1"/>
+<wire x1="12.446" y1="13.716" x2="12.446" y2="13.8684" width="0.1778" layer="1"/>
 <wire x1="12.6238" y1="13.8684" x2="12.446" y2="13.716" width="0.1778" layer="1"/>
 <wire x1="12.6238" y1="13.8684" x2="12.54125" y2="13.81126875" width="0.1778" layer="1"/>
@@
 <wire x1="2.286" y1="15.748" x2="2.286" y2="4.318" width="0.8128" layer="16"/>
 <wire x1="2.286" y1="4.318" x2="5.334" y2="1.27" width="0.8128" layer="16"/>
-<wire x1="11.43" y1="18.8468" x2="12.0904" y2="18.8468" width="0.1778" layer="1"/>
+<wire x1="11.43" y1="18.8468" x2="12.0904" y2="18.8468" width="0.6096" layer="1"/>
 <wire x1="12.0904" y1="18.8468" x2="12.258" y2="18.8261" width="0.1778" layer="1"/>
 <contactref element="TSOC" pad="11B"/>
