File: TSOC_GROVEY_ONE/revisions/R1_1/TSOC_GROVEY_ONE.sch (EAGLE design)
At the start: 49 parts, among them J3 NO, J4 6p-2.54, U1 MIC5219 3.3V, U2 ATMEGA328, X1 16MHZ

Commit message: update to Rev 2.0
Parts:
- R10, R4, R5, R7, R8, R9: value 1K 1/10W -> 1K; device Seeed-Resistor-2016:SMD-RES-1K-5%-1/10W(0603) -> Seeed-Resistor-2016:SMD-RES-2.2K-5%-1/10W(0603)
Changed lines of the file:
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@@
 <setting verticaltext="up"/>
 </settings>
-<grid distance="0.1" unitdist="inch" unit="inch" style="lines" multiple="1" display="no" altdistance="0.01" altunitdist="inch" altunit="inch"/>
+<grid distance="0.1" unitdist="inch" unit="inch" style="dots" multiple="1" display="yes" altdistance="0.01" altunitdist="inch" altunit="inch"/>
 <layers>
 <layer number="1" name="Top" color="4" fill="1" visible="no" active="no"/>
@@
 <part name="UART" library="Seeed-Connector -2016" deviceset="GROVE-CONNECTOR-DIP-90D(4P-2.0)" device="" value="4P-2.0-90D"/>
 <part name="AIO" library="Seeed-Connector -2016" deviceset="GROVE-CONNECTOR-DIP-90D(4P-2.0)" device="" value="4P-2.0-90D"/>
-<part name="R9" library="Seeed-Resistor-2016" deviceset="SMD-RES-1K-5%-1/10W(0603)" device="" value="1K 1/10W"/>
-<part name="R10" library="Seeed-Resistor-2016" deviceset="SMD-RES-1K-5%-1/10W(0603)" device="" value="1K 1/10W"/>
-<part name="R7" library="Seeed-Resistor-2016" deviceset="SMD-RES-1K-5%-1/10W(0603)" device="" value="1K 1/10W"/>
-<part name="R8" library="Seeed-Resistor-2016" deviceset="SMD-RES-1K-5%-1/10W(0603)" device="" value="1K 1/10W"/>
+<part name="R9" library="Seeed-Resistor-2016" deviceset="SMD-RES-2.2K-5%-1/10W(0603)" device="" value="1K"/>
+<part name="R10" library="Seeed-Resistor-2016" deviceset="SMD-RES-2.2K-5%-1/10W(0603)" device="" value="1K"/>
+<part name="R7" library="Seeed-Resistor-2016" deviceset="SMD-RES-2.2K-5%-1/10W(0603)" device="" value="1K"/>
+<part name="R8" library="Seeed-Resistor-2016" deviceset="SMD-RES-2.2K-5%-1/10W(0603)" device="" value="1K"/>
 <part name="R3" library="Seeed-Resistor-2016" deviceset="SMD-RES-2.2K-5%-1/10W(0603)" device="" value="2.2K"/>
 <part name="R2" library="Seeed-Resistor-2016" deviceset="SMD-RES-2.2K-5%-1/10W(0603)" device="" value="2.2K"/>
-<part name="R5" library="Seeed-Resistor-2016" deviceset="SMD-RES-1K-5%-1/10W(0603)" device="" value="1K 1/10W"/>
-<part name="R4" library="Seeed-Resistor-2016" deviceset="SMD-RES-1K-5%-1/10W(0603)" device="" value="1K 1/10W"/>
+<part name="R5" library="Seeed-Resistor-2016" deviceset="SMD-RES-2.2K-5%-1/10W(0603)" device="" value="1K"/>
+<part name="R4" library="Seeed-Resistor-2016" deviceset="SMD-RES-2.2K-5%-1/10W(0603)" device="" value="1K"/>
 <part name="FID4" library="TSOC-ESP8266-BASE" deviceset="FIDUCIAL" device="UFIDUCIAL"/>
 <part name="FID2" library="TSOC-ESP8266-BASE" deviceset="FIDUCIAL" device="UFIDUCIAL"/>

Commit message: update documetation
Parts:
- U1: value MIC5219 3.3V -> AP2112K-3.3V; device TSOC-ESP8266-BASE:V_REG_MIC52193.3V -> SparkFun-PowerIC:V_REG_LDOSMD; PROD_ID (none) -> VREG-12457
Other:
- moved on the sheet: U1
Changed lines of the file:
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@@
 <part name="L1" library="Seeed-Inductor-2016" deviceset="SMD-FERRITE-CHIP-120-OHM-500MA(0603)" device="" value="120OHM-500MA"/>
 <part name="J4" library="Seeed-Connector -2016" deviceset="DIP-BLACK-MALE-HEADER(6P-2.54)" device="" value="6p-2.54"/>
-<part name="U1" library="TSOC-ESP8266-BASE" deviceset="V_REG_MIC5219" device="3.3V" value="MIC5219 3.3V"/>
 <part name="GND7" library="SparkFun" deviceset="GND" device=""/>
 <part name="GND8" library="SparkFun" deviceset="GND" device=""/>
@@
 <part name="GND3" library="supply1" deviceset="GND" device=""/>
 <part name="GND" library="PatternAgents-ProtoPads" deviceset="M01" device="PTH"/>
+<part name="U1" library="SparkFun-PowerIC" deviceset="V_REG_LDO" device="SMD" value="AP2112K-3.3V">
+<attribute name="PROD_ID" value="VREG-12457"/>
+</part>
 </parts>
 <sheets>
@@
 <instance part="L1" gate="L" x="-213.36" y="-91.44"/>
 <instance part="J4" gate="G$1" x="-152.4" y="-44.45"/>
-<instance part="U1" gate="G$1" x="124.46" y="-96.52"/>
 <instance part="GND7" gate="1" x="137.16" y="-119.38"/>
 <instance part="GND8" gate="1" x="109.22" y="-119.38"/>
@@
 <instance part="GND3" gate="1" x="180.34" y="-119.38"/>
 <instance part="GND" gate="G$1" x="195.58" y="-114.3" rot="R180"/>
+<instance part="U1" gate="G$1" x="121.92" y="-96.52">
+<attribute name="PROD_ID" x="121.92" y="-96.52" size="2.54" layer="96" display="off"/>
+</instance>
 </instances>
 <busses>
@@
 </segment>
 <segment>
-<pinref part="U1" gate="G$1" pin="IN"/>
-<wire x1="114.3" y1="-91.44" x2="101.6" y2="-91.44" width="0.1524" layer="91"/>
 <pinref part="C4" gate="G$1" pin="1"/>
-<wire x1="101.6" y1="-105.41" x2="101.6" y2="-96.52" width="0.1524" layer="91"/>
 <label x="187.96" y="-78.74" size="1.27" layer="95" font="vector" ratio="10" xref="yes"/>
-<wire x1="101.6" y1="-96.52" x2="101.6" y2="-91.44" width="0.1524" layer="91"/>
 <wire x1="88.9" y1="-78.74" x2="101.6" y2="-78.74" width="0.1524" layer="91"/>
 <wire x1="101.6" y1="-78.74" x2="149.86" y2="-78.74" width="0.1524" layer="91"/>
 <wire x1="149.86" y1="-78.74" x2="187.96" y2="-78.74" width="0.1524" layer="91"/>
+<wire x1="101.6" y1="-105.41" x2="101.6" y2="-101.6" width="0.1524" layer="91"/>
+<junction x="101.6" y="-78.74"/>
+<wire x1="101.6" y1="-101.6" x2="101.6" y2="-91.44" width="0.1524" layer="91"/>
 <wire x1="101.6" y1="-91.44" x2="101.6" y2="-78.74" width="0.1524" layer="91"/>
-<junction x="101.6" y="-91.44"/>
-<junction x="101.6" y="-78.74"/>
 <wire x1="88.9" y1="-104.14" x2="88.9" y2="-105.41" width="0.1524" layer="91"/>
 <wire x1="88.9" y1="-105.41" x2="88.9" y2="-78.74" width="0.1524" layer="91"/>
 <wire x1="149.86" y1="-81.28" x2="149.86" y2="-78.74" width="0.1524" layer="91"/>
 <junction x="149.86" y="-78.74"/>
-<pinref part="U1" gate="G$1" pin="EN"/>
-<wire x1="114.3" y1="-96.52" x2="101.6" y2="-96.52" width="0.1524" layer="91"/>
-<junction x="101.6" y="-96.52"/>
 <pinref part="J3" gate="JMP" pin="3"/>
 <pinref part="C3" gate="G$1" pin="2"/>
+<pinref part="U1" gate="G$1" pin="EN"/>
+<wire x1="111.76" y1="-101.6" x2="101.6" y2="-101.6" width="0.1524" layer="91"/>
+<junction x="101.6" y="-101.6"/>
+<pinref part="U1" gate="G$1" pin="IN"/>
+<wire x1="111.76" y1="-91.44" x2="101.6" y2="-91.44" width="0.1524" layer="91"/>
+<junction x="101.6" y="-91.44"/>
 </segment>
 </net>
@@
 <segment>
 <pinref part="GND8" gate="1" pin="GND"/>
-<wire x1="109.22" y1="-116.84" x2="109.22" y2="-101.6" width="0.1524" layer="91"/>
+<wire x1="109.22" y1="-116.84" x2="109.22" y2="-96.52" width="0.1524" layer="91"/>
 <pinref part="U1" gate="G$1" pin="GND"/>
-<wire x1="109.22" y1="-101.6" x2="114.3" y2="-101.6" width="0.1524" layer="91"/>
+<wire x1="109.22" y1="-96.52" x2="111.76" y2="-96.52" width="0.1524" layer="91"/>
 </segment>
 <segment>
@@
 <segment>
 <label x="187.96" y="-91.44" size="1.27" layer="95" font="vector" ratio="10" rot="MR180" xref="yes"/>
-<pinref part="U1" gate="G$1" pin="OUT"/>
-<wire x1="132.08" y1="-91.44" x2="149.86" y2="-91.44" width="0.1524" layer="91"/>
 <wire x1="149.86" y1="-91.44" x2="187.96" y2="-91.44" width="0.1524" layer="91"/>
 <junction x="149.86" y="-91.44"/>
@@
 <pinref part="J3" gate="JMP" pin="1"/>
 <pinref part="C5" gate="G$1" pin="2"/>
+<pinref part="U1" gate="G$1" pin="OUT"/>
+<wire x1="149.86" y1="-91.44" x2="129.54" y2="-91.44" width="0.1524" layer="91"/>
 </segment>
 </net>
@@
 <net name="BYPASS1" class="0">
 <segment>
-<pinref part="U1" gate="G$1" pin="BP"/>
-<wire x1="132.08" y1="-101.6" x2="137.16" y2="-101.6" width="0.1524" layer="91"/>
 <wire x1="137.16" y1="-101.6" x2="137.16" y2="-105.41" width="0.1524" layer="91"/>
 <pinref part="C8" gate="G$1" pin="1"/>
-</segment>
-</net>
+<pinref part="U1" gate="G$1" pin="BP"/>
+<wire x1="129.54" y1="-101.6" x2="137.16" y2="-101.6" width="0.1524" layer="91"/>
+</segment>
+</net>
