File: TSOC_GROVEY_ONE/revisions/R2_0/TSOC_GROVEY_ONE.sch (EAGLE design)
At the start: 49 parts, among them J3 NO, J4 6p-2.54, U1 MIC5219 3.3V, U2 ATMEGA328, X1 16MHZ

Commit message: update documetation
Parts:
- removed U1: MIC5219 3.3V, TSOC-ESP8266-BASE:V_REG_MIC52193.3V
- added 5V0: (no value), PatternAgents-ProtoPads:M01PTH
- added U3: AP2112K-3.3V, SparkFun-PowerIC:V_REG_LDOSMD
Connections:
- net 3V3: now also U3.OUT; no longer U1.OUT
- net 5V0: now also 5V0.1, U3.EN, U3.IN; no longer U1.EN, U1.IN
- net BYPASS1: now also U3.BP; no longer U1.BP
- net D0: now also R8.1; no longer R7.1
- net D0E: now also R8.2, UART.1; no longer R7.2, UART.2
- net D1: now also R7.1; no longer R8.1
- net D1E: now also R7.2, UART.2; no longer R8.2, UART.1
- net GND: now also U3.GND; no longer U1.GND
Other:
- moved on the sheet: C11, C3, C4
